File: KiCAD/Mosfets_and_Drivers.sch (KiCad schematic (older format))
At the start: 29 parts, among them P3 CONN_01X01, P4 CONN_01X01, P5 CONN_speaker_plus, P6 CONN_speaker_minus, Q4 Q_NMOS_GDS, Q5 Q_NMOS_GDS, Q6 Q_NMOS_GDS, Q7 Q_NMOS_GDS, U4 ir2010_SOIC, U5 ir2010_SOIC

Commit message: new design for triangular generator
Parts:
- P3, P4, P5, P6: symbol CONN_01X01 -> Conn_01x01
Changed lines of the file:
@@
 EESchema Schematic File Version 2
+LIBS:class_D_ampl-rescue
 LIBS:power
 LIBS:device
@@
 $Descr A4 11693 8268
 encoding utf-8
-Sheet 3 5
+Sheet 3 6
 Title "Mosfets y Drivers"
 Date "2017-02-21"
@@
 $EndComp
 $Comp
-L CONN_01X01 P4
+L Conn_01x01 P4
 U 1 1 58A3490B
 P 6150 1900
@@
 	4650 3500 5850 3500
 $Comp
-L CONN_01X01 P3
+L Conn_01x01 P3
 U 1 1 58A34F5A
 P 6450 5350
@@
 $EndComp
 $Comp
-L CONN_01X01 P5
+L Conn_01x01 P5
 U 1 1 58BEC477
 P 8100 2850
@@
 $EndComp
 $Comp
-L CONN_01X01 P6
+L Conn_01x01 P6
 U 1 1 58BEC673
 P 8150 4700
