File: KiCAD/class_D_ampl.sch (KiCad schematic (older format))
At the start: 1 part, among them P2 BNC

Commit message: change the library for a zener
Parts:
- P2: symbol BNC -> CONN_COAXIAL
Changed lines of the file:
@@
 LIBS:powerint
 LIBS:local
-LIBS:class_D_ampl-cache
 EELAYER 25 0
 EELAYER END
@@
 $EndSheet
 $Comp
-L BNC P2
+L CONN_COAXIAL P2
 U 1 1 58710D34
 P 3400 4000

Commit message: new design for triangular generator
Parts:
- P2: symbol CONN_COAXIAL -> Conn_Coaxial
Changed lines of the file:
@@
 EESchema Schematic File Version 2
+LIBS:class_D_ampl-rescue
 LIBS:power
 LIBS:device
@@
 $Descr A4 11693 8268
 encoding utf-8
-Sheet 1 5
+Sheet 1 6
 Title "Esquéma general"
 Date "2017-02-21"
@@
 $EndSheet
 $Comp
-L CONN_COAXIAL P2
+L Conn_Coaxial P2
 U 1 1 58710D34
 P 3400 4000
@@
 Generador de \nseñal triangular
 $Sheet
-S 1950 3350 1050 950
+S 1550 1500 1050 950
 U 587106D2
 F0 " " 60
 F1 "gen_triangular.sch" 60
-F2 "triangular_signal" O R 3000 3550 60
+F2 "triangular_signal" O R 2600 1700 60
 $EndSheet
 Text Notes 3750 3150 0    120  ~ 0
@@
 Text Notes 8150 3150 0    120  ~ 0
 Drivers y \nMOSFETS de potencia
+$Sheet
+S 1400 3300 1600 1050
+U 5A2D865D
+F0 "generador triangular" 60
+F1 "new_gen_triangular.sch" 60
+F2 "triangular_signal" O R 3000 3550 60
+$EndSheet
 $EndSCHEMATC
