File: KiCAD/gen_triangular.sch (KiCad schematic (older format))
At the start: 20 parts, among them P1 CONN_01X03, Q1 MMBT3904, Q2 MMBT3906, Q3 MMBT3904, Q8 MMBT3906, U1 TLC555

Commit message: change the library for a zener
Parts:
- Z1_3.6V1, Z2_3.6V1: symbol ZENER -> D_Zener_ALT
Changed lines of the file:
@@
 LIBS:powerint
 LIBS:local
-LIBS:class_D_ampl-cache
 EELAYER 25 0
 EELAYER END
@@
 Connection ~ 6600 4050
 $Comp
-L ZENER Z2_3.6V1
+L D_Zener_ALT Z2_3.6V1
 U 1 1 583A2109
 P 7650 4750
@@
 $EndComp
 $Comp
-L ZENER Z1_3.6V1
+L D_Zener_ALT Z1_3.6V1
 U 1 1 583A2324
 P 7650 3450
@@
 	7400 4350 7850 4350
 Wire Wire Line
-	7650 4550 7650 4350
+	7650 4350 7650 4600
 Connection ~ 7650 4350
 $Comp
@@
 $EndComp
 Wire Wire Line
-	7650 5050 7650 4950
-Wire Wire Line
-	7650 3650 7650 3750
+	7650 4900 7650 5050
+Wire Wire Line
+	7650 3600 7650 3750
 Wire Wire Line
 	7400 3750 7850 3750
@@
 $EndComp
 Wire Wire Line
-	7650 3250 7650 3150
+	7650 3150 7650 3300
 Wire Wire Line
 	8150 2850 8150 2800

Commit message: new design for triangular generator
Parts:
- P1: symbol CONN_01X03 -> Conn_01x03
Changed lines of the file:
@@
 EESchema Schematic File Version 2
+LIBS:class_D_ampl-rescue
 LIBS:power
 LIBS:device
@@
 $Descr A4 11693 8268
 encoding utf-8
-Sheet 5 5
+Sheet 5 6
 Title "Generador de señal triangular"
 Date "2017-02-21"
@@
 $EndComp
 $Comp
-L CONN_01X03 P1
+L Conn_01x03 P1
 U 1 1 58A33689
 P 1500 1450
